Commit message: Task 1 Complete: Add controllers and Gazebo simulation
- Added ros2_control configuration with GazeboSimSystem plugin
- Configured joint limits: ±2π for all joints except elbow (±π)
- Added joint_state_broadcaster, forward_position_controller, joint_trajectory_controller
- Created Gazebo launch file with table, cube, and robot spawn
- Fixed Gazebo integration to use direct gz sim command
- Installed required dependencies: gz-harmonic, ros-gz packages, controllers

File: src/ur3_description/urdf/ur3.ros2_control.xacro (robot description, xacro)
@@ -2,10 +2,62 @@
 <robot xmlns:xacro="http://ros.org/wiki/xacro">
   <xacro:macro name="ur3_ros2_control" params="name prefix">
+    <ros2_control name="${name}" type="system">
+      <hardware>
+        <plugin>gz_ros2_control/GazeboSimSystem</plugin>
+      </hardware>
+      <joint name="${prefix}shoulder_pan_joint">
+        <command_interface name="position">
+          <param name="min">-6.2832</param>
+          <param name="max">6.2832</param>
+        </command_interface>
+        <state_interface name="position"/>
+        <state_interface name="velocity"/>
+      </joint>
+      <joint name="${prefix}shoulder_lift_joint">
+        <command_interface name="position">
+          <param name="min">-6.2832</param>
+          <param name="max">6.2832</param>
+        </command_interface>
+        <state_interface name="position"/>
+        <state_interface name="velocity"/>
+      </joint>
+      <joint name="${prefix}elbow_joint">
+        <command_interface name="position">
+          <param name="min">-3.1416</param>
+          <param name="max">3.1416</param>
+        </command_interface>
+        <state_interface name="position"/>
+        <state_interface name="velocity"/>
+      </joint>
+      <joint name="${prefix}wrist_1_joint">
+        <command_interface name="position">
+          <param name="min">-6.2832</param>
+          <param name="max">6.2832</param>
+        </command_interface>
+        <state_interface name="position"/>
+        <state_interface name="velocity"/>
+      </joint>
+      <joint name="${prefix}wrist_2_joint">
+        <command_interface name="position">
+          <param name="min">-6.2832</param>
+          <param name="max">6.2832</param>
+        </command_interface>
+        <state_interface name="position"/>
+        <state_interface name="velocity"/>
+      </joint>
+      <joint name="${prefix}wrist_3_joint">
+        <command_interface name="position">
+          <param name="min">-6.2832</param>
+          <param name="max">6.2832</param>
+        </command_interface>
+        <state_interface name="position"/>
+        <state_interface name="velocity"/>
+      </joint>
+    </ros2_control>
     <gazebo>
-      <!-- add plugin info here -->
+      <plugin filename="gz_ros2_control-system" name="gz_ros2_control::GazeboSimROS2ControlPlugin">
+        <parameters>$(find ur3_description)/config/ur3_controllers.yaml</parameters>
+      </plugin>
     </gazebo>
-    <ros2_control name="${name}" type="system">
-      <!-- add controller info here -->
-    </ros2_control>
   </xacro:macro>
 </robot>
